File: plutopack_frontend_pcb/plutopack/power_management.kicad_sch (KiCad schematic)
At the start: 70 parts, among them J3 Battery_Cell, J5 USB_C_Receptacle_PowerOnly_6P, Q1 AO3401A, Q2 AO3400A, Q3 AO3400A, Q4 AO3401A, SW10 SW_SPDT, U1 BQ24075RGT, U3 TPS63020, U4 BQ27441-G1, U5 TPS63020, U6 BQ297xy

Commit message: Update frontend PCB to latest revision
Sync plutopack_frontend_pcb with the latest KiCad layout, power_management
schematic changes, and regenerated JLC production outputs (BOM, positions,
netlist, gerber zip).

Co-Authored-By: Claude Opus 5.5 (1M context) <noreply@anthropic.com>
Parts:
- added D9: LED, LED_SMD:LED_0603_1608Metric, symbol Device:LED
- added R58: 1k, Resistor_SMD:R_0603_1608Metric, symbol Device:R
Connections:
- net GND: now also D9.1 (K)
- net VCC: now also R58.2
- new net: D9.2 (A), R58.1
